File: Hadware/9axis_minimal/9axis_minimal.sch (KiCad schematic (older format))
At the start: 49 parts, among them J1 Batt, J2 uC_TTL, J3 I2C, J4 panel, J5 USB_C, J7 RTC, Q1 PN2222A, Q2 IRLML6402, Q3 2N3904, SW1 uC_boot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

Commit message: hardware
Parts:
- removed R?: 47R, Resistor_SMD:R_1206_3216Metric_Pad1.30x1.75mm_HandSolder, symbol Device:R_Small
Connections:
- net +3V3: now also BZ1.1 (-)
Changed lines of the file:
@@
 L power:+3.3V #PWR02
 U 1 1 60602B48
-P 1750 4950
-F 0 "#PWR02" H 1750 4800 50  0001 C CNN
-F 1 "+3.3V" H 1765 5123 50  0000 C CNN
-F 2 "" H 1750 4950 50  0001 C CNN
-F 3 "" H 1750 4950 50  0001 C CNN
-	1    1750 4950
+P 1750 5150
+F 0 "#PWR02" H 1750 5000 50  0001 C CNN
+F 1 "+3.3V" H 1765 5323 50  0000 C CNN
+F 2 "" H 1750 5150 50  0001 C CNN
+F 3 "" H 1750 5150 50  0001 C CNN
+	1    1750 5150
 	1    0    0    -1
 $EndComp
@@
 Text GLabel 1000 5650 0    50   Input ~ 0
 Buzzer
-$Comp
-L Device:R_Small R?
-U 1 1 60590A4B
-P 1750 5050
-F 0 "R?" H 1950 5100 50  0000 R CNN
-F 1 "47R" H 2000 5000 50  0000 R CNN
-F 2 "Resistor_SMD:R_1206_3216Metric_Pad1.30x1.75mm_HandSolder" H 1750 5050 50  0001 C CNN
-F 3 "~" H 1750 5050 50  0001 C CNN
-	1    1750 5050
-	-1   0    0    -1
-$EndComp
 $EndSCHEMATC
