File: Hadware/fullaxis_receptor/fullaxis_receptor.kicad_pcb (KiCad board)
At the start: 2 copper layers, 38 parts, among them J1 Batt, J2 uC_TTL, J3 I2C, J4 panel, J5 USB_C, J7 RTC, Q3 2N3904, U1 GY-BNO055, U3 uSD, U4 AMS1117-3.3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

Commit message: hardware
Parts:
- removed BZ1: Buzzer, Buzzer_Beeper:MagneticBuzzer_PUI_AT-0927-TT-6-R
- removed C10, C7: 10uF, Capacitor_SMD:C_1206_3216Metric_Pad1.33x1.80mm_HandSolder
- removed C11: 100nF, Capacitor_SMD:C_1206_3216Metric_Pad1.33x1.80mm_HandSolder
- removed C12, C13, C14: 0.1uF, Capacitor_SMD:C_1206_3216Metric_Pad1.33x1.80mm_HandSolder
- removed C5, C6: 1uF, Capacitor_SMD:C_1206_3216Metric_Pad1.33x1.80mm_HandSolder
- removed C8: 10nF, Capacitor_SMD:C_1206_3216Metric_Pad1.33x1.80mm_HandSolder
- removed J2: uC_TTL, Connector_JST:JST_GH_BM06B-GHS-TBT_1x06-1MP_P1.25mm_Vertical
- removed J3: I2C, Connector_JST:JST_GH_BM04B-GHS-TBT_1x04-1MP_P1.25mm_Vertical
- removed J4: panel, Connector_JST:JST_GH_BM06B-GHS-TBT_1x06-1MP_P1.25mm_Vertical
- removed J5: USB_C, Connector_JST:JST_GH_BM05B-GHS-TBT_1x05-1MP_P1.25mm_Vertical
- removed J7: RTC, Connector_JST:JST_GH_BM05B-GHS-TBT_1x05-1MP_P1.25mm_Vertical
- removed Q3: 2N3904, Package_TO_SOT_THT:TO-92_Inline
- removed R13: 10k, Resistor_SMD:R_1206_3216Metric_Pad1.30x1.75mm_HandSolder
- removed R5: 0.4R, Resistor_SMD:R_1206_3216Metric_Pad1.30x1.75mm_HandSolder
- removed R6: 1.2k, Resistor_SMD:R_1206_3216Metric_Pad1.30x1.75mm_HandSolder
- removed R7: 1M, Resistor_SMD:R_1206_3216Metric_Pad1.30x1.75mm_HandSolder
- removed R8: 100K, Resistor_SMD:R_1206_3216Metric_Pad1.30x1.75mm_HandSolder
- removed R9: 0R, Resistor_SMD:R_1206_3216Metric_Pad1.30x1.75mm_HandSolder
- removed U3: uSD, Connector_JST:JST_GH_BM06B-GHS-TBT_1x06-1MP_P1.25mm_Vertical
- removed U4: AMS1117-3.3, Package_TO_SOT_SMD:SOT-223-3_TabPin2
- removed U6: CH340C, Package_SO:SOIC-16_3.9x9.9mm_P1.27mm
- added SW1: uC_boot, Switches:TACTILE_SWITCH_SMD_6.0X3.5MM, F.Cu at (78.3, 77.7)
- added SW2: uC_reset, Switches:TACTILE_SWITCH_SMD_6.0X3.5MM, F.Cu at (88.2, 77.7)
- added U2: AMS1117-3.3, Package_TO_SOT_SMD:SOT-223-3_TabPin2, F.Cu at (80.1, 90.1)
- C1, C4: value 10uF -> 22nF
- C2: value 10uF -> 100nF; footprint Capacitor_SMD:C_1206_3216Metric_Pad1.33x1.80mm_HandSolder -> Capacitor_SMD:C_1210_3225Metric_Pad1.33x2.70mm_HandSolder
- C3: footprint Capacitor_SMD:C_1206_3216Metric_Pad1.33x1.80mm_HandSolder -> Capacitor_SMD:C_1210_3225Metric_Pad1.33x2.70mm_HandSolder
- J1: value Batt -> USB_A; footprint Connector_JST:JST_GH_BM03B-GHS-TBT_1x03-1MP_P1.25mm_Vertical -> Connector_USB:USB_A_CONNFLY_DS1095-WNR0
- R1: value 1k -> 10K
- R2: value 100k -> 10K
- U1: value GY-BNO055 -> ch340n; footprint Connector_PinSocket_2.54mm:PinSocket_1x08_P2.54mm_Horizontal -> ch340:SOIC-10
- moved C4 61.1 mm to (80.1, 95.5), turned to 180 degrees
- moved C9 56.8 mm to (76.7, 72.9), turned to 180 degrees
- moved R11 55.2 mm to (84.3, 72.9)
- moved R10 44.1 mm to (79.3, 81.0)
- moved R2 43.1 mm to (89.9, 72.9), turned to 180 degrees
- moved R1 43.0 mm to (84.8, 82.2), turned to 90 degrees
- moved U1 36.6 mm to (88.0, 99.7)
- moved R12 36.3 mm to (89.8, 81.0)
- moved C2 32.5 mm to (89.2, 87.8)
- moved J1 30.0 mm to (79.8, 105.7)
- moved C1 28.2 mm to (80.1, 84.8)
- moved U5 24.0 mm to (83.3, 58.1)
- moved C3 20.8 mm to (89.2, 91.6)
Connections:
- C1 pad 1: +BATT -> GND
- C1 pad 2: GND -> +5V
- C2 pad 1: Net-(C2-Pad1) -> +5V
- C3 pad 1: Batt_current -> +3V3
- C4 pad 1: +BATT -> GND
- C4 pad 2: GND -> +3V3
- J1 pad 1: GND -> +5V
- J1 pad 2: +BATT -> D-
- J1 pad 3: NTC -> D+
- R1 pad 1: Net-(Q3-Pad1) -> +3V3
- R1 pad 2: Buzzer -> Net-(R1-Pad2)
- R2 pad 1: Net-(Q3-Pad1) -> Net-(R2-Pad1)
- U1 pad 1: +3V3 -> D+
- U1 pad 2: GND -> D-
- U1 pad 3: SCL -> GND
- U1 pad 4: SDA -> unconnected-(U1-Pad4)
- U1 pad 5: unconnected-(U1-Pad5) -> +3V3
- U1 pad 6: INT_BNO -> uC_RX
- U1 pad 7: unconnected-(U1-Pad7) -> uC_TX
- U1 pad 8: unconnected-(U1-Pad8) -> +3V3
- U5 pad 10: MISO -> unconnected-(U5-Pad10)
- U5 pad 11: unconnected-(U5-Pad11) -> Net-(R1-Pad2)
- U5 pad 12: SS -> unconnected-(U5-Pad12)
- U5 pad 13: MOSI -> unconnected-(U5-Pad13)
- U5 pad 14: SCLK -> unconnected-(U5-Pad14)
- U5 pad 16: uC_SDIO -> Net-(R2-Pad1)
- U5 pad 19: SDA -> unconnected-(U5-Pad19)
- U5 pad 2: Batt_current -> unconnected-(U5-Pad2)
- U5 pad 20: SCL -> unconnected-(U5-Pad20)
- U5 pad 4: SS1 -> unconnected-(U5-Pad4)
- U5 pad 5: Buzzer -> unconnected-(U5-Pad5)
- U5 pad 6: auto_pwr -> unconnected-(U5-Pad6)
- U5 pad 7: INT_BNO -> unconnected-(U5-Pad7)
Routing:
- net GND: track 0.00 -> 68.4 mm
- net +3V3: track 0.00 -> 63.8 mm
- net uC_reset: track 0.00 -> 62.6 mm
- net uC_RX: track 0.00 -> 49.5 mm
- net uC_TX: track 0.00 -> 48.6 mm
- net uC_boot: track 0.00 -> 44.7 mm
- net +5V: track 0.00 -> 23.0 mm
- net Net-(R1-Pad2): track 0.00 -> 20.2 mm
- net Net-(R11-Pad2): track 0.00 -> 18.9 mm
- net Net-(R2-Pad1): track 0.00 -> 9.68 mm
- net D-: track 0.00 -> 8.86 mm
- net D+: track 0.00 -> 3.91 mm
- added copper zone on F.Cu, net GND
